File: BB Call Call back/BB Call/layout/BB Call/BB Call.kicad_sch (KiCad schematic)
At the start: 52 parts, among them J1 104031-0811, P2 USB_C_Plug_USB2.0, Q2 S8050, Q3 S8050, U10 CH340C, U11 AMS1117, U12 USBLC6-2SC6, U13 ESP32-S3, U15 W25Q128JV, U16 APS1604M-3SQRx-SN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

Commit message: Update the battery
Update the battery
Other:
- added sheet Battery (Battery.kicad_sch)
Changed lines of the file:
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@@
+	)
+	(sheet
+		(at 223.52 104.14)
+		(size 50.8 33.02)
+		(exclude_from_sim no)
+		(in_bom yes)
+		(on_board yes)
+		(dnp no)
+		(fields_autoplaced yes)
+		(stroke
+			(width 0.1524)
+			(type solid)
+		)
+		(fill
+			(color 0 0 0 0)
+		)
+		(property "Sheetname" "Battery"
+			(at 223.52 103.4284 0)
+			(show_name no)
+			(do_not_autoplace no)
+			(effects
+				(font
+					(size 1.27 1.27)
+				)
+				(justify left bottom)
+			)
+		)
+		(property "Sheetfile" "Battery.kicad_sch"
+			(at 223.52 137.7446 0)
+			(show_name no)
+			(do_not_autoplace no)
+			(effects
+				(font
+					(size 1.27 1.27)
+				)
+				(justify left top)
+			)
+		)
+		(instances
+			(project "BB Call"
+				(path "/e866ee95-ac75-4662-818c-95723bb4362d"
+					(page "2")
+				)
+			)
+		)
 	)
 	(sheet
